File: ESP07_Tool.sch (EAGLE design)
At the start: 53 parts

Commit message: Update for pogo changes
Parts:
- removed 3V3_, ADC, CH_PD, GND, GND_, GPIO0, GPIO12, GPIO13, GPIO14, GPIO15, GPIO16, GPIO2, GPIO4, GPIO5, REST, RXD, RXD_, TXD, TXD_, VCC: (no value), wirepad:SMD2
- added U$3: SMD-PAD-SM, CuriousTech:SMD-PAD-SM
- added U$4, U$5, U$6, U$7: SMD-PAD1, CuriousTech:SMD-PAD1
- U$1: value SMD-PAD-SM -> ESP-07/12; device CuriousTech:SMD-PAD-SM -> ESP-07_12:ESP-07/12
Connections:
- net 3V3: now also U$1.P$9, U$6.P$1; no longer 3V3_.P, VCC.P
- net GND: now also U$1.P$8, U$7.P$1; no longer GND.P, GND_.P
- net N$10: now also U$1.P$5; no longer GPIO0.P
- net N$11: now also U$1.P$14; no longer CH_PD.P
- net N$12: now also U$1.P$15; no longer ADC.P
- net N$15: now also U$1.P$13; no longer GPIO16.P
- net N$16: now also U$1.P$12; no longer GPIO14.P
- net N$17: now also U$1.P$11; no longer GPIO12.P
- net N$18: now also U$1.P$10; no longer GPIO13.P
- net N$22: now also U$1.P$16; no longer REST.P
- net N$3: now also U$1.P$3; no longer GPIO4.P
- net N$7: now also U$1.P$6; no longer GPIO2.P
- net N$8: now also U$1.P$7; no longer GPIO15.P
- net N$9: now also U$1.P$4; no longer GPIO5.P
- net RXD: now also U$1.P$2, U$4.P$1; no longer RXD.P, RXD_.P
- net TXD: now also U$1.P$1, U$5.P$1; no longer TXD.P, TXD_.P
- net VCC: now also U$3.P$1; no longer U$1.P$1
Other:
- moved on the sheet: C3, C7, C8, FLASH, IO2, JP1, R1, R2, R3, R6, RUN
